Commit message: launchable robot arm

File: urdf/ur3e_robot.urdf (robot description, URDF)
Before this commit: robot ur3e_robot, 13 links, 12 joints
Links:
- link base_link_inertia: geometry visual mesh filename=../meshes/ur3e/visual/base.dae
- link forearm_link: geometry visual mesh filename=../meshes/ur3e/visual/forearm.dae
- link shoulder_link: geometry visual mesh filename=../meshes/ur3e/visual/shoulder.dae
- link upper_arm_link: geometry visual mesh filename=../meshes/ur3e/visual/upperarm.dae
- link wrist_1_link: geometry visual mesh filename=../meshes/ur3e/visual/wrist1.dae
- link wrist_2_link: geometry visual mesh filename=../meshes/ur3e/visual/wrist2.dae
- link wrist_3_link: geometry visual mesh filename=../meshes/ur3e/visual/wrist3.dae
