Commit message: Patch: use multibody for visualization only

File: resources/bicopter.urdf (robot description, URDF)
Before this commit: robot bicopter, 5 links, 4 joints
Links:
- link body: mass None -> 1
- link propeller_left: mass None -> 1
- link propeller_right: mass None -> 1
- link propguard_left: mass None -> 1
- link propguard_right: mass None -> 1
